File: schematics/board/SPin.sch (EAGLE design)
At the start: 15 parts

Commit message: Добавлены платы SP
Connections:
- removed net GND: R14.2, U$13.S
- net BUS-: now also R14.2, U$13.S
Changed lines of the file:
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@@
 <wire x1="73.66" y1="25.4" x2="58.42" y2="25.4" width="0.1524" layer="91"/>
 </segment>
-</net>
-<net name="GND" class="0">
 <segment>
 <pinref part="U$13" gate="G$1" pin="S"/>
