File: schematics/board/SPin.brd (EAGLE design)
At the start: 71.4 x 71.4 mm, 15 parts

Commit message: Добавлены платы SP
Connections:
- removed net GND: R14.2, U$13.2
- net BUS-: now also R14.2, U$13.2
Routing:
- net GND: track 4.12 -> 0.00 mm
- net BUS-: track 0.00 -> 4.12 mm, vias 0 -> 1
Changed lines of the file:
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@@
 <vertex x="40.7" y="64.7"/>
 </polygon>
-</signal>
-<signal name="GND">
 <contactref element="U$13" pad="2"/>
 <contactref element="R14" pad="2"/>
-<wire x1="26.05" y1="61.45" x2="28.4" y2="61.45" width="0.5" layer="1"/>
-<wire x1="28.4" y1="61.45" x2="29.65" y2="62.7" width="0.5" layer="1"/>
+<wire x1="29.65" y1="62.7" x2="28.4" y2="61.45" width="1" layer="1"/>
+<wire x1="26.05" y1="61.45" x2="28.4" y2="61.45" width="1" layer="1"/>
+<via x="28.4" y="61.45" extent="1-16" drill="0.35"/>
 </signal>
 <signal name="ROZE">
